File: PCB/tycharlie-lily58.kicad_pcb (KiCad board)
At the start: 2 copper layers, 146.4 x 104.4 mm, 78 parts, among them J1 Conn_01x02_Pin, J2 Conn_01x05_Pin, J3 AudioJack4, SW1 SW_Push, SW10 SW_Push, SW11 SW_Push, SW12 SW_Push, SW13 SW_Push, SW14 SW_Push, SW15 SW_Push, SW16 SW_Push, SW17 SW_Push, SW18 SW_Push, SW19 SW_Push, SW2 SW_Push, SW20 SW_Push, SW21 SW_Push, SW22 SW_Push, SW23 SW_Push, SW24 SW_Push, SW25 SW_Push, SW26 SW_Push, SW27 SW_Push, SW28 SW_Push, SW29 SW_Push, SW3 SW_Push, SW30 SW_Push, SW4 SW_Push, SW5 SW_Push, SW6 SW_Push, SW7 SW_Push, SW8 SW_Push, SW9 SW_Push, U1 SuperMini nRF52840

Commit message: CHORE: add the name on pcb
Parts:
- SW30: moved to F.Cu
Other:
- board text added: "By TsungYu"

Commit message: FIX: update the battery footprint
  - Add new Molex PicoBlade 53261 foorprint
  - Changed the battery pin1 to BATT+
Parts:
- J1: footprint tycharlie-lily58:JST_GH_SM02B-GHS-TB_1x02-1MP_P1.25mm_Horizontal -> tycharlie-lily58:Molex_PicoBlade_53261-0271_1x02-1MP_P1.25mm_Horizontal
- moved J1 11.2 mm to (200.1, 78.0)
Connections:
- J1 pad 1: GND -> +BATT
- J1 pad 2: +BATT -> GND
Routing:
- net +BATT: track 93.2 -> 105.3 mm
